Commit message: Update robot data

File: urdf/n_v1.urdf (robot description, URDF)
Before this commit: robot simple_diff_drive, 3 links, 2 joints
Links:
- link base_link: geometry visual box size=0.3 0.3 0.015
- link left_wheel: geometry visual cylinder length=0.042 radius=0.055
- link right_wheel: geometry visual cylinder length=0.042 radius=0.055
Joints:
- joint left_wheel_joint: origin xyz=0 -0.15 0 rpy=0 0 0 -> xyz=0 -0.15 0.055 rpy=0 0 0

Commit message: Add imu link definition

File: urdf/n_v1.urdf (robot description, URDF)
Before this commit: robot n1_diff_drive, 3 links, 2 joints
Links:
- added link imu_link
Joints:
- added joint base_to_imu: type fixed, parent base_link, child imu_link, origin xyz=0.0 0.0 0.0 rpy=0.0 0.0 0.0

Commit message: Add visual components of imu link

File: urdf/n_v1.urdf (robot description, URDF)
Before this commit: robot n1_diff_drive, 4 links, 3 joints
Links:
- link imu_link: mass None -> 0.0492; geometry visual box size=0.054 0.054 0.0189

Commit message: Add laser link definition

File: urdf/n_v1.urdf (robot description, URDF)
Before this commit: robot n1_diff_drive, 4 links, 3 joints
Links:
- added link laser_link; visual cylinder length=0.07 radius=0.038
Joints:
- added joint base_to_laser: type fixed, parent base_link, child laser_link, origin xyz=0.092 0 0.151 rpy=0 0 0

Commit message: Add base footprint definition

File: urdf/n_v1.urdf (robot description, URDF)
Before this commit: robot n1_diff_drive, 5 links, 4 joints
Links:
- added link base_footprint; visual box size=0.3 0.3 0.10
- link base_link: geometry visual box size=0.3 0.3 0.10
Joints:
- added joint base_footprint_to_base_link: type fixed, parent base_link, child base_footprint, origin xyz=0 0 0 rpy=0 0 0

Commit message: Fix origin component of right_wheel and imu joint

File: urdf/n_v1.urdf (robot description, URDF)
Before this commit: robot n1_diff_drive, 6 links, 5 joints
Joints:
- joint base_to_imu: origin xyz=0.0 0.0 0.0 rpy=0.0 0.0 0.0 -> xyz=-0.045 0.105 0.10 rpy=0.0 0.0 1.57079
- joint right_wheel_joint: origin xyz=0 0.15 0 rpy=0 0 0 -> xyz=0 0.15 0.055 rpy=0 0 0

Commit message: Fix origin component of imu joint

File: urdf/n_v1.urdf (robot description, URDF)
Before this commit: robot n1_diff_drive, 6 links, 5 joints
Joints:
- joint base_to_imu: origin xyz=-0.045 0.105 0.10 rpy=0.0 0.0 1.57079 -> xyz=-0.045 0.105 0.10 rpy=0.0 0.0 -1.57079

Commit message: Temporarily change origin component of imu joint

File: urdf/n_v1.urdf (robot description, URDF)
Before this commit: robot n1_diff_drive, 6 links, 5 joints
Joints:
- joint base_to_imu: origin xyz=-0.045 0.105 0.10 rpy=0.0 0.0 -1.57079 -> xyz=0 0 0 rpy=0.0 0.0 -1.57079

Commit message: Temporarily change origin component of laser joint

File: urdf/n_v1.urdf (robot description, URDF)
Before this commit: robot n1_diff_drive, 6 links, 5 joints
Joints:
- joint base_to_laser: origin xyz=0.092 0 0.151 rpy=0 0 0 -> xyz=0.092 0 0.151 rpy=0 0 3.14179
